Commit message: refactor: decouple TurtleBot3 Lime packages from Gazebo

File: turtlebot3_lime_description/urdf/materials.urdf.xacro (robot description, xacro)
@@ -1,8 +1,5 @@
-<?xml version="1.0"?>
-<!--
-Copied from open_manipulator example -
-https://github.com/ROBOTIS-GIT/open_manipulator/blob/foxy-devel/open_manipulator_x_description/urdf/materials.xacro
--->
-<robot>
+<?xml version="1.0" ?>
+<robot name="materials"
+  xmlns:xacro="http://ros.org/wiki/xacro">
   <material name="black">
     <color rgba="0.0 0.0 0.0 1.0"/>

File: turtlebot3_lime_hardware/ros2_control/turtlebot3_lime.urdf.xacro (robot description, xacro)
@@ -10,4 +10,6 @@
   <!-- Include OpenManipulator-X urdf macro -->
   <xacro:include filename="$(find turtlebot3_lime_description)/urdf/open_manipulator_sara.urdf.xacro" />
+  <!-- Include ROS 2 Control urdf macro -->
+  <xacro:include filename="$(find turtlebot3_lime_hardware)/ros2_control/turtlebot3_lime_system.ros2_control.xacro" />
   <xacro:turtlebot3_bigwheel_orin prefix="$(arg prefix)" />
   <!-- Fixed joint between the mobile base and manipulator -->
@@ -18,3 +20,8 @@
   </joint>
   <xacro:open_manipulator_sara prefix="$(arg prefix)" />
+  <xacro:turtlebot3_lime_system
+    name="TurtleBot3LimeSystem"
+    prefix="$(arg prefix)"
+    use_fake_hardware="$(arg use_fake_hardware)"
+    fake_sensor_commands="$(arg fake_sensor_commands)" />
 </robot>

File: turtlebot3_lime_hardware/ros2_control/turtlebot3_lime_system.ros2_control.xacro (robot description, xacro)
@@ -6,30 +6,25 @@
 -->
 <robot xmlns:xacro="http://www.ros.org/wiki/xacro">
-  <xacro:macro name="turtlebot3_lime_system" params="name prefix use_sim:=^|false use_fake_hardware:=^|false fake_sensor_commands:=^|false">
+  <xacro:macro
+    name="turtlebot3_lime_system"
+    params="name prefix use_fake_hardware:=^|false fake_sensor_commands:=^|false">
     <ros2_control name="${name}" type="system">
-      <xacro:if value="$(arg use_sim)">
-        <hardware>
-          <plugin>gazebo_ros2_control/GazeboSystem</plugin>
-        </hardware>
-      </xacro:if>
-      <xacro:unless value="$(arg use_sim)">
-        <hardware>
-          <xacro:if value="${use_fake_hardware}">
-            <plugin>fake_components/GenericSystem</plugin>
-            <param name="fake_sensor_commands">${fake_sensor_commands}</param>
-            <param name="state_following_offset">0.0</param>
-          </xacro:if>
-          <xacro:unless value="${use_fake_hardware}">
-            <plugin>turtlebot3_lime_hardware/TurtleBot3LimeSystemHardware</plugin>
-            <param name="opencr_id">200</param>
-            <param name="opencr_usb_port">/dev/ttyACM0</param>
-            <param name="opencr_baud_rate">1000000</param>
-            <param name="dxl_joints_profile_acceleration">100</param>
-            <param name="dxl_joints_profile_velocity">500</param>
-            <param name="dxl_gripper_profile_acceleration">20</param>
-            <param name="dxl_gripper_profile_velocity">200</param>
-          </xacro:unless>
-        </hardware>
-      </xacro:unless>
+      <hardware>
+        <xacro:if value="${use_fake_hardware}">
+          <plugin>fake_components/GenericSystem</plugin>
+          <param name="fake_sensor_commands">${fake_sensor_commands}</param>
+          <param name="state_following_offset">0.0</param>
+        </xacro:if>
+        <xacro:unless value="${use_fake_hardware}">
+          <plugin>turtlebot3_lime_hardware/TurtleBot3LimeSystemHardware</plugin>
+          <param name="opencr_id">200</param>
+          <param name="opencr_usb_port">/dev/ttyACM0</param>
+          <param name="opencr_baud_rate">1000000</param>
+          <param name="dxl_joints_profile_acceleration">100</param>
+          <param name="dxl_joints_profile_velocity">500</param>
+          <param name="dxl_gripper_profile_acceleration">20</param>
+          <param name="dxl_gripper_profile_velocity">200</param>
+        </xacro:unless>
+      </hardware>
       <joint name="${prefix}wheel_left_joint">
         <command_interface name="velocity">
