Commit message: update

File: turtlebot3_lime_description/urdf/control/turtlebot3_lime_system.ros2_control.xacro (robot description, xacro)
@@ -197,4 +197,25 @@
       </joint>
     </ros2_control>
+    <xacro:if value="${use_gazebo}">
+      <gazebo>
+        <plugin
+          filename="gz_ros2_control-system"
+          name="gz_ros2_control::GazeboSimROS2ControlPlugin">
+          <robot_param>robot_description</robot_param>
+          <robot_param_node>robot_state_publisher</robot_param_node>
+          <parameters>
+            $(find turtlebot3_lime_gazebo)/config/ros2_controllers.yaml
+          </parameters>
+          <ros>
+            <remapping>
+              /diff_drive_controller/cmd_vel_unstamped:=/cmd_vel
+            </remapping>
+            <remapping>
+              /diff_drive_controller/odom:=/odom
+            </remapping>
+          </ros>
+        </plugin>
+      </gazebo>
+    </xacro:if>
   </xacro:macro>
 </robot>

File: turtlebot3_lime_gazebo/urdf/sensors/imu.gazebo.xacro (robot description, xacro)
@@ -11,4 +11,5 @@
         <visualize>false</visualize>
         <topic>imu</topic>
+        <gz_frame_id>${prefix}imu_link</gz_frame_id>
       </sensor>
     </gazebo>

File: turtlebot3_lime_gazebo/urdf/sensors/lidar.gazebo.xacro (robot description, xacro)
@@ -12,4 +12,5 @@
         <visualize>true</visualize>
         <topic>scan</topic>
+        <gz_frame_id>${prefix}base_scan</gz_frame_id>
         <lidar>
           <scan>

File: turtlebot3_lime_gazebo/urdf/sensors/rgbd_camera.gazebo.xacro (robot description, xacro)
@@ -10,4 +10,5 @@
         <visualize>true</visualize>
         <topic>camera</topic>
+        <gz_frame_id>${prefix}camera_link</gz_frame_id>
         <camera>
           <horizontal_fov>1.2112585008840648</horizontal_fov>

File: turtlebot3_lime_gazebo/urdf/turtlebot3_bigwheel_orin.gazebo.xacro (robot description, xacro)
@@ -2,9 +2,9 @@
 <robot xmlns:xacro="http://www.ros.org/wiki/xacro">
   <xacro:include
-    filename="$(find turtlebot3_lime_gazebo)/urdf/sensors/imu.gazebo.xacro"/>
+    filename="$(find turtlebot3_lime_gazebo)/urdf/sensors/imu.gazebo.xacro" />
   <xacro:include
-    filename="$(find turtlebot3_lime_gazebo)/urdf/sensors/lidar.gazebo.xacro"/>
+    filename="$(find turtlebot3_lime_gazebo)/urdf/sensors/lidar.gazebo.xacro" />
   <xacro:include
-    filename="$(find turtlebot3_lime_gazebo)/urdf/sensors/rgbd_camera.gazebo.xacro"/>
+    filename="$(find turtlebot3_lime_gazebo)/urdf/sensors/rgbd_camera.gazebo.xacro" />
   <xacro:macro name="turtlebot3_bigwheel_orin_gazebo" params="prefix">
     <gazebo reference="${prefix}base_link">
@@ -14,10 +14,18 @@
       <mu1>1.0</mu1>
       <mu2>1.0</mu2>
-      <material>Gazebo/Green</material>
+      <material>
+        <ambient>0.0 0.8 0.0 1.0</ambient>
+        <diffuse>0.0 0.8 0.0 1.0</diffuse>
+        <specular>0.1 0.1 0.1 1.0</specular>
+      </material>
     </gazebo>
     <gazebo reference="${prefix}wheel_right_link">
       <mu1>1.0</mu1>
       <mu2>1.0</mu2>
-      <material>Gazebo/Green</material>
+      <material>
+        <ambient>0.0 0.8 0.0 1.0</ambient>
+        <diffuse>0.0 0.8 0.0 1.0</diffuse>
+        <specular>0.1 0.1 0.1 1.0</specular>
+      </material>
     </gazebo>
     <gazebo reference="${prefix}caster_back_right_link">
@@ -32,9 +40,9 @@
     </gazebo>
     <xacro:turtlebot3_lime_imu_gazebo
-      prefix="${prefix}"/>
+      prefix="${prefix}" />
     <xacro:turtlebot3_lime_lidar_gazebo
-      prefix="${prefix}"/>
+      prefix="${prefix}" />
     <xacro:turtlebot3_lime_rgbd_camera_gazebo
-      prefix="${prefix}"/>
+      prefix="${prefix}" />
   </xacro:macro>
 </robot>

File: turtlebot3_lime_gazebo/urdf/turtlebot3_lime.urdf.xacro (robot description, xacro)
@@ -7,11 +7,15 @@
   <xacro:include filename="$(find turtlebot3_lime_description)/urdf/materials.urdf.xacro" />
   <!-- Include TurtleBot3 BigWheel Orin URDF macro -->
-  <xacro:include filename="$(find turtlebot3_lime_description)/urdf/turtlebot3_bigwheel_orin.urdf.xacro" />
+  <xacro:include
+    filename="$(find turtlebot3_lime_description)/urdf/turtlebot3_bigwheel_orin.urdf.xacro" />
   <!-- Include OpenManipulator-X urdf macro -->
-  <xacro:include filename="$(find turtlebot3_lime_description)/urdf/open_manipulator_sara.urdf.xacro" />
+  <xacro:include
+    filename="$(find turtlebot3_lime_description)/urdf/open_manipulator_sara.urdf.xacro" />
   <!-- Include TurtleBot3 Lime System urdf macro -->
-  <xacro:include filename="$(find turtlebot3_lime_description)/urdf/control/turtlebot3_lime_system.ros2_control.xacro"/>
+  <xacro:include
+    filename="$(find turtlebot3_lime_description)/urdf/control/turtlebot3_lime_system.ros2_control.xacro" />
   <!-- Include TurtleBot3 BigWheel Orin Gazebo macro -->
-  <xacro:include filename="$(find turtlebot3_lime_gazebo)/urdf/turtlebot3_bigwheel_orin.gazebo.xacro" />
+  <xacro:include
+    filename="$(find turtlebot3_lime_gazebo)/urdf/turtlebot3_bigwheel_orin.gazebo.xacro" />
   <!-- Include OpenManipulator SARA Gazebo macro -->
   <xacro:include filename="$(find turtlebot3_lime_gazebo)/urdf/open_manipulator_sara.gazebo.xacro" />
@@ -19,9 +23,10 @@
   <!-- Fixed joint between the mobile base and manipulator -->
   <joint name="$(arg prefix)base_fixed" type="fixed">
-    <parent link="$(arg prefix)base_link"/>
-    <child link="$(arg prefix)link1"/>
-    <origin xyz="-0.036 0.0 0.07" rpy="0 0 0"/>
+    <parent link="$(arg prefix)base_link" />
+    <child link="$(arg prefix)link1" />
+    <origin xyz="-0.036 0.0 0.07" rpy="0 0 0" />
   </joint>
-  <xacro:open_manipulator_sara prefix="$(arg prefix)" />
+  <!-- Reduced simulation friction: effort limits are 1 N m (arm) and 1 N (gripper). -->
+  <xacro:open_manipulator_sara prefix="$(arg prefix)" arm_friction="0.01" gripper_friction="0.01" />
   <xacro:turtlebot3_bigwheel_orin_gazebo prefix="$(arg prefix)" />
   <xacro:open_manipulator_sara_gazebo prefix="$(arg prefix)" />
@@ -31,4 +36,4 @@
     use_gazebo="true"
     use_fake_hardware="false"
-    fake_sensor_commands="false"/>
+    fake_sensor_commands="false" />
 </robot>
